File: hw_modules/dc_servor_driver/hw/control_board.sch (KiCad schematic (older format))
At the start: 33 parts, among them P1 CONN_02X03, P2 CONN_01X06, P3 CONN_01X03, P4 CONN_02X03, Q1 BSS138, Q4 BSS138, Q5 BSS138, Q6 BSS138, Q7 BSS138, U1 STM32F030F4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

Commit message: Firt verision of dc_servo_driver board
Parts:
- removed C6: 470n, Capacitors_SMD:C_0603, symbol C_Small
- removed C7: 100n, Capacitors_SMD:C_0603, symbol C_Small
- removed P2: CONN_01X06, Pin_Headers:Pin_Header_Angled_1x06, symbol CONN_01X06
- removed Q1, Q4, Q5, Q6, Q7: BSS138, TO_SOT_Packages_SMD:SOT-23, symbol BSS138
- removed R10, R11, R12, R13, R14, R15, R16: 10k, Resistors_SMD:R_0603, symbol R
- removed U2: APE8865N-33-HF-3, TO_SOT_Packages_SMD:SOT-23, symbol APE8865N-33-HF-3
- added R6: 10k, Resistors_SMD:R_0603, symbol R
- added R7, R9: 20k, Resistors_SMD:R_0603, symbol R
- added U2: FDI_Module_Half, yaqwsx:FTDI_Half, symbol FDI_Module_Half
- R5: value 10k -> 20k
- Y1: value 8Mhz -> Crystal_Four_Pin
Connections:
- net labels added: UART_CTS, UART_RTS, UART_RX, UART_TX
- net labels removed: UART_RX_3.3, UART_RX_5, UART_TX_3.3, UART_TX_5
- wire segments 102 -> 50
- no-connect marks 8 -> 14
Other:
- moved on the sheet: C2
