File: hw_modules/spindle_light/spindle_light.sch (KiCad schematic (older format))
At the start: 81 parts

Commit message: Add missing files for spindle light
Parts:
- gave numbers to parts that had none: 1
