File: hw_modules/old_dc_servo_driver/hw/vykonova deska.sch (EAGLE design)
At the start: 23 parts, among them IC1 HCPL-3120, Q1 IRG4PC50W, Q2 IRG4PC50W

Commit message: Add PWM to -+10V board
Parts:
- D2, D3: value 15A10G -> STTH15R06D
Changed lines of the file:
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@@
 <?xml version="1.0" encoding="utf-8"?>
 <!DOCTYPE eagle SYSTEM "eagle.dtd">
-<eagle version="7.2.0">
+<eagle version="9.0.1">
 <drawing>
 <settings>
 <setting alwaysvectorfont="no"/>
+<setting keepoldvectorfont="yes"/>
 <setting verticaltext="up"/>
 </settings>
@@
 <part name="SUPPLY2" library="supply2" deviceset="GND" device=""/>
 <part name="C1" library="resistor" deviceset="C-EU" device="102-043X133" value="10n 1kV"/>
-<part name="D3" library="adafruit" deviceset="1N4004" device="" value="15A10G"/>
+<part name="D3" library="adafruit" deviceset="1N4004" device="" value="STTH15R06D"/>
 <part name="C2" library="resistor" deviceset="C-EU" device="102-043X133" value="10n 1kV"/>
 <part name="C3" library="resistor" deviceset="C-EU" device="C0603" value="100n"/>
@@
 <part name="R6" library="resistor" deviceset="R-EU_" device="R0603" value="330R"/>
 <part name="X2" library="con-wago-508" deviceset="W237-2N" device=""/>
-<part name="D2" library="adafruit" deviceset="1N4004" device="" value="15A10G"/>
+<part name="D2" library="adafruit" deviceset="1N4004" device="" value="STTH15R06D"/>
 <part name="X1" library="con-wago-508" deviceset="W237-3N" device=""/>
 <part name="SUPPLY5" library="supply2" deviceset="VCC" device="" value="+180V"/>
