File: hw_modules/spindle_h_bridge/half-bridge.sch (KiCad schematic (older format))
At the start: 24 parts, among them Q1 IRG4PH40U, Q2 IRG4PH40U, U4 FAN7393A

Commit message: Add PWM to -+10V board
Parts:
- C5: footprint Capacitors_SMD:C_1206 -> Capacitor_SMD:C_1206_3216Metric_Pad1.42x1.75mm_HandSolder; symbol C -> spindle_h_bridge-rescue:C
- C6: footprint Capacitors_SMD:C_0603 -> Capacitor_SMD:C_0603_1608Metric_Pad1.05x0.95mm_HandSolder; symbol C -> spindle_h_bridge-rescue:C
- C7, C8: footprint Capacitors_ThroughHole:C_Rect_L7_W4.5_P5 -> Capacitor_THT:C_Rect_L7.0mm_W4.5mm_P5.00mm; symbol C -> spindle_h_bridge-rescue:C
- C9: footprint Capacitors_ThroughHole:C_Rect_L10_W6_P7.5 -> Capacitor_THT:C_Rect_L7.0mm_W4.5mm_P5.00mm; symbol C -> spindle_h_bridge-rescue:C
- D1, D2: footprint Diodes_ThroughHole:Diode_TO-220_Vertical -> Package_TO_SOT_THT:TO-220-2_Vertical; symbol D_Schottky -> spindle_h_bridge-rescue:D_Schottky
- D10, D11, D7: footprint Diodes_SMD:SOD-323 -> Diode_SMD:D_SOD-323_HandSoldering; symbol BAT42 -> spindle_h_bridge-rescue:BAT42
- D13, D9: footprint Diodes_SMD:MELF_Standard -> Diode_SMD:D_MELF_Handsoldering; symbol D_Zener -> spindle_h_bridge-rescue:D_Zener
- Q1, Q2: footprint TO_SOT_Packages_THT:TO-247_Vertical_Neutral123 -> Package_TO_SOT_THT:TO-247-3_Horizontal_TabDown; symbol Q_NIGBT_GCE -> spindle_h_bridge-rescue:Q_NIGBT_GCE
- R11, R12, R13, R14, R3, R4, R5: footprint Resistors_SMD:R_0603 -> Resistor_SMD:R_0603_1608Metric_Pad1.05x0.95mm_HandSolder; symbol R -> spindle_h_bridge-rescue:R
- R15, R16: footprint Resistors_ThroughHole:Resistor_Horizontal_RM10mm -> Resistor_THT:R_Box_L14.0mm_W5.0mm_P9.00mm; symbol R -> spindle_h_bridge-rescue:R
- U4: footprint Housings_SOIC:SOIC-14_3.9x8.7mm_Pitch1.27mm -> Package_SO:SOIC-14_3.9x8.7mm_P1.27mm; symbol FAN7393A -> yaqwsx:FAN7393A
