File: hw_modules/spindle_h_bridge/spindle_h_bridge.sch (KiCad schematic (older format))
At the start: 14 parts, among them J1 SIGNAL, J2 MOTOR, J3 POWER, J4 POWER, U1 ADuM1200AR, U2 LM1117-5.0

Commit message: Add PWM to -+10V board
Parts:
- added H1, H2, H3, H4: MountingHole, MountingHole:MountingHole_3.2mm_M3, symbol Mechanical:MountingHole
- C1: footprint Capacitors_SMD:C_1206 -> Capacitor_SMD:C_1206_3216Metric_Pad1.42x1.75mm_HandSolder; symbol C -> spindle_h_bridge-rescue:C
- C15, C17: footprint Capacitors_SMD:C_1206 -> Capacitor_SMD:C_0603_1608Metric_Pad1.05x0.95mm_HandSolder; symbol C -> spindle_h_bridge-rescue:C
- C16, C18: footprint Capacitors_SMD:C_0603 -> Capacitor_SMD:C_0603_1608Metric_Pad1.05x0.95mm_HandSolder; symbol C -> spindle_h_bridge-rescue:C
- C19: footprint Capacitors_SMD:c_elec_4x4.5 -> Capacitor_SMD:CP_Elec_4x4.5; symbol CP -> spindle_h_bridge-rescue:CP
- C3, C4: footprint Capacitors_ThroughHole:C_Radial_D16_L25_P7.5 -> Capacitor_THT:CP_Radial_D16.0mm_P7.50mm; symbol CP -> spindle_h_bridge-rescue:CP
- J1: footprint Terminal_Blocks:TerminalBlock_Pheonix_MKDS1.5-4pol -> TerminalBlock_Phoenix:TerminalBlock_Phoenix_MKDS-1,5-4_1x04_P5.00mm_Horizontal; symbol CONN_01X04 -> spindle_h_bridge-rescue:CONN_01X04
- J2, J3, J4: footprint Terminal_Blocks:TerminalBlock_Pheonix_MKDS1.5-2pol -> TerminalBlock_Phoenix:TerminalBlock_Phoenix_MKDS-1,5-2_1x02_P5.00mm_Horizontal; symbol CONN_01X02 -> spindle_h_bridge-rescue:CONN_01X02
- U1: footprint Housings_SOIC:SOIC-8_3.9x4.9mm_Pitch1.27mm -> Package_SO:SOIC-8_3.9x4.9mm_P1.27mm; symbol ADuM1200AR -> spindle_h_bridge-rescue:ADuM1200AR
- U2: footprint TO_SOT_Packages_SMD:SOT-223 -> Package_TO_SOT_SMD:SOT-223; symbol LM1117-5.0 -> spindle_h_bridge-rescue:LM1117-5.0
Connections:
- net left-half-bridge/OUT: now also J2.1 (P1); no longer J2.2 (P2)
- net left-half-bridge/PWM: now also U1.6 (VOB); no longer U1.7 (VOA)
- net right-half-bridge/OUT: now also J2.2 (P2); no longer J2.1 (P1)
- net right-half-bridge/PWM: now also U1.7 (VOA); no longer U1.6 (VOB)
